File: eagle/ver2_usb/team4-selo-atmega32u4-usb.brd (EAGLE design)
At the start: 62 x 40 mm, 35 parts, among them J1 3x2 M, J3 629105136821, SW2 !RESET, U3 ATMEGA32U4-AUR, X2 16 MHz

Commit message: edit board layout file
Parts:
- moved H1 30.0 mm to (87.0, 37.0)
- moved H3 30.0 mm to (87.0, 3.00)
- moved NUMPAD 27.2 mm to (86.0, 19.0)
Routing:
- net N$6: track 0.00 -> 68.6 mm, vias 0 -> 2
- net N$11: track 0.00 -> 56.8 mm, vias 0 -> 2
- net N$10: track 0.00 -> 51.4 mm, vias 0 -> 2
- net N$5: track 0.00 -> 49.0 mm, vias 0 -> 2
- net N$2: track 0.00 -> 46.9 mm, vias 0 -> 1
- net N$9: track 0.00 -> 45.2 mm, vias 0 -> 2
- net N$8: track 0.00 -> 42.8 mm, vias 0 -> 2
- net N$12: track 0.00 -> 42.5 mm, vias 0 -> 1
- net N$21: track 3.51 -> 44.0 mm, vias 1 -> 2
- net VBUS: track 103.3 -> 115.2 mm
- net TX_LED: track 34.2 -> 36.0 mm, vias 1 -> 2
Other:
- board size 62 x 40 mm -> 90 x 40 mm

Commit message: reroute on eagle board, update gitignore
Parts:
- moved SERVO 31.8 mm to (56.0, 6.00)
- moved H1 25.3 mm to (62.0, 33.0)
- moved H3 25.0 mm to (62.0, 3.00)
- moved NUMPAD 24.0 mm to (62.0, 19.0)
- moved H2 4.00 mm to (3.00, 33.0)
- moved C16 3.00 mm to (35.8, 4.10)
- moved C17 3.00 mm to (43.4, 4.10)
- moved X2 3.00 mm to (39.6, 7.90)
- moved C11 2.24 mm to (36.1, 12.6)
- moved D3 1.18 mm to (51.9, 31.0)
- moved C3 1.00 mm to (51.3, 19.8)
Routing:
- net N$10: track 51.4 -> 18.2 mm
- net N$6: track 68.6 -> 38.5 mm, vias 2 -> 6
- net N$9: track 45.2 -> 18.7 mm, vias 2 -> 1
- net N$12: track 42.5 -> 18.5 mm, vias 1 -> 0
- net N$5: track 49.0 -> 25.1 mm, vias 2 -> 4
- net N$8: track 42.8 -> 18.8 mm
- net N$1: track 45.4 -> 22.7 mm, vias 0 -> 2
- net N$11: track 56.8 -> 34.5 mm
- net N$2: track 46.9 -> 26.7 mm
- net GND: track 34.4 -> 21.2 mm, vias 0 -> 4
- net N$21: track 44.0 -> 40.7 mm, vias 2 -> 1
- net TX_LED: track 36.0 -> 34.4 mm
- net VBUS: track 115.2 -> 116.7 mm, vias 1 -> 4
- net N$17: track 52.8 -> 54.2 mm
- net XTAL2: track 14.7 -> 15.9 mm
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Other:
- board size 90 x 40 mm -> 65 x 36 mm

Commit message: update eagle board
Routing:
- net VBUS: track 116.7 -> 128.4 mm
- net N$6: vias 6 -> 5
- net N$11: vias 2 -> 1
Changed lines of the file:
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@@
 <drawing>
 <settings>
-<setting alwaysvectorfont="yes"/>
+<setting alwaysvectorfont="no"/>
 <setting keepoldvectorfont="yes"/>
 <setting verticaltext="up"/>
@@
 <layers>
 <layer number="1" name="Top" color="4" fill="1" visible="yes" active="yes"/>
-<layer number="2" name="Route2" color="1" fill="3" visible="no" active="yes"/>
+<layer number="2" name="Route2" color="1" fill="3" visible="yes" active="yes"/>
 <layer number="15" name="Route15" color="4" fill="6" visible="no" active="yes"/>
 <layer number="16" name="Bottom" color="1" fill="1" visible="yes" active="yes"/>
@@
 <contactref element="U3" pad="15"/>
 <contactref element="U3" pad="5"/>
-<polygon width="0.254" layer="1">
+<polygon width="0.254" layer="1" isolate="0.254">
 <vertex x="0" y="0"/>
 <vertex x="65" y="0"/>
@@
 <vertex x="0" y="36"/>
 </polygon>
-<polygon width="0.254" layer="16">
+<polygon width="0.254" layer="16" isolate="0.254">
 <vertex x="0" y="0"/>
 <vertex x="65" y="0"/>
@@
 <wire x1="34.29" y1="24.892" x2="34.29" y2="24.79998125" width="0.254" layer="1"/>
 <via x="38" y="15" extent="1-16" drill="0.35"/>
-<via x="48" y="18" extent="1-16" drill="0.35"/>
+<via x="46" y="19" extent="1-16" drill="0.35"/>
 <via x="43" y="34" extent="1-16" drill="0.35"/>
 <via x="31.3" y="24.8" extent="1-16" drill="0.35"/>
@@
 <contactref element="C19" pad="1"/>
 <contactref element="U3" pad="2"/>
-<wire x1="34.2" y1="27.2" x2="10.5" y2="27.2" width="0.5" layer="1"/>
+<wire x1="34.2" y1="27.2" x2="30" y2="27.2" width="0.5" layer="1"/>
+<wire x1="30" y1="27.2" x2="10.5" y2="27.2" width="0.5" layer="1"/>
 <wire x1="9.1" y1="28.6" x2="10.5" y2="27.2" width="0.5" layer="1"/>
-<wire x1="4.075" y1="25.3" x2="6.2" y2="25.3" width="0.4" layer="1"/>
-<wire x1="6.2" y1="25.3" x2="8" y2="27.1" width="0.4" layer="1"/>
-<wire x1="8" y1="27.1" x2="8" y2="28.4" width="0.5" layer="1"/>
-<wire x1="8" y1="28.4" x2="8" y2="28.6" width="0.4" layer="1"/>
 <wire x1="8" y1="28.6" x2="9.1" y2="28.6" width="0.5" layer="1"/>
-<wire x1="8.05" y1="28.45" x2="8" y2="28.4" width="0.4" layer="1"/>
 <contactref element="SERVO" pad="2"/>
 <contactref element="U3" pad="44"/>
@@
 <contactref element="R8" pad="2"/>
 <contactref element="R12" pad="2"/>
-<wire x1="35.814" y1="29.718" x2="36" y2="29.8" width="0.254" layer="1"/>
-<wire x1="43.942" y1="29.718" x2="44" y2="29.8" width="0.254" layer="1"/>
 <wire x1="56" y1="17" x2="52.2" y2="20.8" width="0.5" layer="1"/>
 <wire x1="52.2" y1="20.8" x2="51.3" y2="20.8" width="0.5" layer="1"/>
@@
 <wire x1="44" y1="31" x2="44" y2="29.8" width="0.5" layer="1"/>
 <wire x1="56" y1="6" x2="56" y2="17" width="0.5" layer="1"/>
-<wire x1="34.2" y1="27.2" x2="34.2" y2="29.8" width="0" layer="19" extent="1-1"/>
-<wire x1="34.2" y1="23.2" x2="34.2" y2="27.2" width="0" layer="19" extent="1-1"/>
+<wire x1="4.075" y1="25.3" x2="6.3" y2="25.3" width="0.4" layer="1"/>
+<wire x1="6.3" y1="25.3" x2="8" y2="27" width="0.4" layer="1"/>
+<wire x1="8" y1="27" x2="8" y2="28.6" width="0.4" layer="1"/>
+<wire x1="34.2" y1="29.8" x2="30.8" y2="29.8" width="0.5" layer="1"/>
+<wire x1="30.8" y1="29.8" x2="30" y2="29" width="0.5" layer="1"/>
+<wire x1="30" y1="29" x2="30" y2="27.2" width="0.5" layer="1"/>
+<wire x1="34.2" y1="27.2" x2="35.8" y2="27.2" width="0.5" layer="1"/>
+<wire x1="35.8" y1="27.2" x2="36" y2="27" width="0.5" layer="1"/>
+<wire x1="36" y1="27" x2="36" y2="23.2" width="0.5" layer="1"/>
 </signal>
 <signal name="N$19">
 <contactref element="J3" pad="2"/>
 <contactref element="R4" pad="1"/>
-<wire x1="4.075" y1="24.65" x2="8.25" y2="24.65" width="0.4" layer="1"/>
-<wire x1="8.25" y1="24.65" x2="9" y2="25.4" width="0.4" layer="1"/>
-<wire x1="9" y1="25.4" x2="10.15" y2="25.4" width="0.4" layer="1"/>
+<wire x1="4.075" y1="24.65" x2="8.25" y2="24.65" width="0.3" layer="1"/>
+<wire x1="8.25" y1="24.65" x2="9" y2="25.4" width="0.3" layer="1"/>
+<wire x1="9" y1="25.4" x2="10.15" y2="25.4" width="0.3" layer="1"/>
 </signal>
 <signal name="N$20">
 <contactref element="J3" pad="3"/>
 <contactref element="R5" pad="1"/>
-<wire x1="4.075" y1="24" x2="8.3" y2="24" width="0.4" layer="1"/>
-<wire x1="8.3" y1="24" x2="9.1" y2="23.2" width="0.4" layer="1"/>
-<wire x1="9.1" y1="23.2" x2="10.15" y2="23.2" width="0.4" layer="1"/>
+<wire x1="4.075" y1="24" x2="8.3" y2="24" width="0.3" layer="1"/>
+<wire x1="8.3" y1="24" x2="9.1" y2="23.2" width="0.3" layer="1"/>
+<wire x1="9.1" y1="23.2" x2="10.15" y2="23.2" width="0.3" layer="1"/>
 </signal>
 <signal name="D+">
@@
 <via x="54.9335625" y="23.932" extent="1-16" drill="0.35"/>
 <wire x1="60" y1="18.8655625" x2="60" y2="16" width="0.3" layer="16"/>
-<via x="60" y="16" extent="1-16" drill="0.35"/>
 <wire x1="57.2924375" y1="23.706" x2="57.706" y2="23.2924375" width="0.3" layer="16"/>
 <wire x1="54.9335625" y1="23.932" x2="55.1595625" y2="23.706" width="0.3" layer="16"/>
@@
 <wire x1="57.706" y1="21.1595625" x2="60" y2="18.8655625" width="0.3" layer="16"/>
 <wire x1="57.706" y1="23.2924375" x2="57.706" y2="21.1595625" width="0.3" layer="16"/>
-<wire x1="60" y1="16" x2="60.81" y2="15.19" width="0.3" layer="1"/>
-<wire x1="60.81" y1="15.19" x2="62" y2="15.19" width="0.3" layer="1"/>
+<wire x1="60" y1="16" x2="60.81" y2="15.19" width="0.3" layer="16"/>
+<wire x1="60.81" y1="15.19" x2="62" y2="15.19" width="0.3" layer="16"/>
 </signal>
 <signal name="N$1">
@@
 <wire x1="49.1842625" y1="27.8157375" x2="51" y2="26" width="0.3" layer="16"/>
 <wire x1="51" y1="26" x2="59" y2="26" width="0.3" layer="16"/>
-<via x="59" y="26" extent="1-16" drill="0.35"/>
-<wire x1="59" y1="26" x2="59.65" y2="25.35" width="0.3" layer="1"/>
-<wire x1="59.65" y1="25.35" x2="62" y2="25.35" width="0.3" layer="1"/>
+<wire x1="59" y1="26" x2="59.65" y2="25.35" width="0.3" layer="16"/>
+<wire x1="59.65" y1="25.35" x2="62" y2="25.35" width="0.3" layer="16"/>
 </signal>
 <signal name="N$12">
@@
 <contactref element="U3" pad="19"/>
 <contactref element="BUZZER" pad="1"/>
-<wire x1="41.6" y1="18.2" x2="41.746" y2="18.054" width="0.3" layer="1"/>
 <wire x1="41.656" y1="19.05" x2="41.656" y2="18.288" width="0.254" layer="1"/>
 <wire x1="42.164" y1="19.558" x2="41.656" y2="19.05" width="0.254" layer="1"/>

Commit message: check with DRC
Routing:
- net VBUS: track 128.4 -> 130.9 mm
Changed lines of the file:
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@@
 <wire x1="9" y1="5.27" x2="14.54" y2="5.27" width="0.3" layer="1"/>
 <wire x1="14.54" y1="5.27" x2="15" y2="5.73" width="0.3" layer="1"/>
-<wire x1="34.29" y1="24.892" x2="34.2" y2="24.8" width="0.254" layer="1"/>
-<wire x1="34.29" y1="24.892" x2="34.29" y2="24.79998125" width="0.254" layer="1"/>
 <via x="38" y="15" extent="1-16" drill="0.35"/>
 <via x="46" y="19" extent="1-16" drill="0.35"/>
@@
 <wire x1="45.8" y1="20.8" x2="38" y2="20.8" width="0.5" layer="1"/>
 <wire x1="38" y1="20.8" x2="37.6" y2="20.4" width="0.5" layer="1"/>
-<wire x1="36" y1="29.8" x2="36" y2="31" width="0.5" layer="1"/>
-<via x="36" y="31" extent="1-16" drill="0.35"/>
-<wire x1="36" y1="31" x2="44" y2="31" width="0.5" layer="16"/>
-<via x="44" y="31" extent="1-16" drill="0.35"/>
-<wire x1="44" y1="31" x2="44" y2="29.8" width="0.5" layer="1"/>
+<wire x1="36" y1="29.8" x2="36" y2="32" width="0.5" layer="1"/>
+<via x="36" y="32" extent="1-16" drill="0.35"/>
+<wire x1="44" y1="32" x2="36" y2="32" width="0.5" layer="16"/>
+<via x="44" y="32" extent="1-16" drill="0.35"/>
+<wire x1="44" y1="32" x2="44" y2="29.8" width="0.5" layer="1"/>
 <wire x1="56" y1="6" x2="56" y2="17" width="0.5" layer="1"/>
-<wire x1="4.075" y1="25.3" x2="6.3" y2="25.3" width="0.4" layer="1"/>
-<wire x1="6.3" y1="25.3" x2="8" y2="27" width="0.4" layer="1"/>
-<wire x1="8" y1="27" x2="8" y2="28.6" width="0.4" layer="1"/>
 <wire x1="34.2" y1="29.8" x2="30.8" y2="29.8" width="0.5" layer="1"/>
 <wire x1="30.8" y1="29.8" x2="30" y2="29" width="0.5" layer="1"/>
@@
 <wire x1="35.8" y1="27.2" x2="36" y2="27" width="0.5" layer="1"/>
 <wire x1="36" y1="27" x2="36" y2="23.2" width="0.5" layer="1"/>
+<wire x1="4.075" y1="25.3" x2="5.3" y2="25.3" width="0.4" layer="1"/>
+<wire x1="5.3" y1="25.3" x2="6" y2="26" width="0.4" layer="1"/>
+<wire x1="6" y1="26" x2="8" y2="26" width="0.4" layer="1"/>
+<wire x1="8" y1="26" x2="8" y2="28.6" width="0.4" layer="1"/>
 </signal>
 <signal name="N$19">
@@
 </signal>
 <signal name="N$22">
-<via x="36" y="33" extent="1-16" drill="0.35"/>
+<via x="35" y="34" extent="1-16" drill="0.35"/>
 </signal>
 <signal name="N$24">
@@
 <mfgpreviewcolor name="substratecolor" color="0xFF786E46"/>
 </mfgpreviewcolors>
+<errors>
+</errors>
 </board>
 </drawing>
