File: eagle/ver2_usb/team4-selo-atmega32u4-usb.brd (EAGLE design)
At the start: 65 x 36 mm, 35 parts, among them J1 3x2 M, J3 629105136821, SW2 !RESET, U3 ATMEGA32U4-AUR, X2 16 MHz

Commit message: update board and schematic
Parts:
- moved BUZZER 4.12 mm to (14.0, 11.0)
Connections:
- removed net N$3: R3.2
- net VBUS: now also R3.2
Routing:
- net VBUS: track 130.9 -> 138.2 mm
- net N$21: track 40.5 -> 34.7 mm
- net GND: track 20.9 -> 23.4 mm, vias 4 -> 11
Other:
- board text added: "Team 4 - version#1 SeLo - Security Locker 11/19/2019"
- board text removed: "Team 4 - version#1 SeLo - Security Locker"
Changed lines of the file:
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@@
 <drawing>
 <settings>
-<setting alwaysvectorfont="no"/>
+<setting alwaysvectorfont="yes"/>
 <setting keepoldvectorfont="yes"/>
 <setting verticaltext="up"/>
@@
 <layers>
 <layer number="1" name="Top" color="4" fill="1" visible="yes" active="yes"/>
-<layer number="2" name="Route2" color="1" fill="3" visible="yes" active="yes"/>
+<layer number="2" name="Route2" color="1" fill="3" visible="no" active="yes"/>
 <layer number="15" name="Route15" color="4" fill="6" visible="no" active="yes"/>
 <layer number="16" name="Bottom" color="1" fill="1" visible="yes" active="yes"/>
@@
 <wire x1="65" y1="36" x2="0" y2="36" width="0" layer="20"/>
 <wire x1="0" y1="36" x2="0" y2="0" width="0" layer="20"/>
-<text x="8" y="32" size="0.6096" layer="21" font="vector" ratio="20">ECE411 32u4 Board Rev 1
-Based on Arduino Lilypad Rev 10
-CC by-SA</text>
-<text x="15" y="30" size="0.6096" layer="21" font="vector">Team 4 - version#1
-SeLo - Security Locker</text>
+<text x="5" y="15" size="0.4064" layer="21" font="vector" ratio="20">ECE411 32u4 Board Rev 1
+Based on Arduino Lilypad
+Rev 10 CC by-SA</text>
+<text x="15" y="31" size="0.8128" layer="21" font="vector">Team 4 - version#1
+SeLo - Security Locker
+11/19/2019</text>
 </plain>
 <attributes>
@@
 <attribute name="VALUE" x="58.825" y="29.16" size="1.27" layer="27" rot="R270"/>
 </element>
-<element name="BUZZER" library="pinhead" library_urn="urn:adsk.eagle:library:325" package="1X02" package3d_urn="urn:adsk.eagle:package:22435/2" value="" x="15" y="7" smashed="yes" rot="R270">
-<attribute name="NAME" x="16.8288" y="9.6162" size="1.27" layer="25" ratio="10" rot="R270"/>
-<attribute name="POPULARITY" value="98" x="15" y="7" size="1.778" layer="27" rot="R270" display="off"/>
-<attribute name="VALUE" x="11.825" y="9.54" size="1.27" layer="27" rot="R270"/>
+<element name="BUZZER" library="pinhead" library_urn="urn:adsk.eagle:library:325" package="1X02" package3d_urn="urn:adsk.eagle:package:22435/2" value="" x="14" y="11" smashed="yes" rot="R270">
+<attribute name="NAME" x="15.8288" y="13.6162" size="1.27" layer="25" ratio="10" rot="R270"/>
+<attribute name="POPULARITY" value="98" x="14" y="11" size="1.778" layer="27" rot="R270" display="off"/>
+<attribute name="VALUE" x="10.825" y="13.54" size="1.27" layer="27" rot="R270"/>
 </element>
 <element name="LEDS" library="pinhead" library_urn="urn:adsk.eagle:library:325" package="1X02" package3d_urn="urn:adsk.eagle:package:22435/2" value="" x="9" y="4" smashed="yes" rot="R90">
@@
 <wire x1="9" y1="5.27" x2="3.4" y2="10.87" width="0.3" layer="1"/>
 <wire x1="3.4" y1="10.87" x2="3.4" y2="17.7" width="0.3" layer="1"/>
-<wire x1="9" y1="5.27" x2="14.54" y2="5.27" width="0.3" layer="1"/>
-<wire x1="14.54" y1="5.27" x2="15" y2="5.73" width="0.3" layer="1"/>
+<wire x1="9" y1="5.27" x2="12.54" y2="5.27" width="0.3" layer="1"/>
+<wire x1="14" y1="6.73" x2="14" y2="9.73" width="0.3" layer="1"/>
+<wire x1="14" y1="6.73" x2="12.54" y2="5.27" width="0.3" layer="1"/>
 <via x="38" y="15" extent="1-16" drill="0.35"/>
-<via x="46" y="19" extent="1-16" drill="0.35"/>
+<via x="47" y="19" extent="1-16" drill="0.35"/>
 <via x="43" y="34" extent="1-16" drill="0.35"/>
 <via x="31.3" y="24.8" extent="1-16" drill="0.35"/>
+<via x="32" y="12" extent="1-16" drill="0.35"/>
+<via x="35" y="34" extent="1-16" drill="0.35"/>
+<via x="50" y="31" extent="1-16" drill="0.35"/>
+<via x="10" y="10" extent="1-16" drill="0.35"/>
+<via x="10" y="20" extent="1-16" drill="0.35"/>
+<via x="55" y="2" extent="1-16" drill="0.35"/>
+<via x="13" y="31" extent="1-16" drill="0.35"/>
 </signal>
 <signal name="!RESET">
@@
 <wire x1="6" y1="26" x2="8" y2="26" width="0.4" layer="1"/>
 <wire x1="8" y1="26" x2="8" y2="28.6" width="0.4" layer="1"/>
+<contactref element="R3" pad="2"/>
+<wire x1="22.15" y1="16.15" x2="22.15" y2="13.85" width="0.5" layer="1"/>
+<wire x1="23.8" y1="12.2" x2="26.45" y2="12.2" width="0.5" layer="1"/>
+<wire x1="22.15" y1="13.85" x2="23.8" y2="12.2" width="0.5" layer="1"/>
 </signal>
 <signal name="N$19">
@@
 <wire x1="44.45" y1="22.606" x2="44.958" y2="23.114" width="0.254" layer="1"/>
 <wire x1="44.45" y1="21.59" x2="44.45" y2="22.606" width="0.254" layer="1"/>
-<wire x1="44.45" y1="19.558" x2="44.45" y2="21.59" width="0.254" layer="16"/>
-<wire x1="44.45" y1="19.558" x2="48.768" y2="15.24" width="0.254" layer="16"/>
+<wire x1="44.45" y1="19.558" x2="44.45" y2="21.59" width="0.3" layer="16"/>
+<wire x1="44.45" y1="19.558" x2="48.768" y2="15.24" width="0.3" layer="16"/>
 <wire x1="45.72" y1="23.114" x2="45.8" y2="23.2" width="0.254" layer="1"/>
 <via x="44.45" y="21.59" extent="1-16" drill="0.254"/>
@@
 <contactref element="U3" pad="19"/>
 <contactref element="BUZZER" pad="1"/>
-<wire x1="41.656" y1="19.05" x2="41.656" y2="18.288" width="0.254" layer="1"/>
-<wire x1="42.164" y1="19.558" x2="41.656" y2="19.05" width="0.254" layer="1"/>
-<wire x1="44.196" y1="19.558" x2="42.164" y2="19.558" width="0.254" layer="1"/>
-<wire x1="44.704" y1="19.05" x2="44.196" y2="19.558" width="0.254" layer="1"/>
-<wire x1="44.704" y1="16.764" x2="44.704" y2="19.05" width="0.254" layer="1"/>
-<wire x1="44.704" y1="16.51" x2="44.704" y2="16.764" width="0.254" layer="16"/>
-<wire x1="38.608" y1="10.414" x2="44.704" y2="16.51" width="0.254" layer="16"/>
-<wire x1="16.256" y1="10.414" x2="38.608" y2="10.414" width="0.254" layer="16"/>
-<wire x1="14.986" y1="9.144" x2="16.256" y2="10.414" width="0.254" layer="16"/>
-<wire x1="14.986" y1="8.382" x2="14.986" y2="9.144" width="0.254" layer="16"/>
-<wire x1="41.656" y1="18.288" x2="41.6" y2="18.2" width="0.254" layer="1"/>
-<wire x1="14.986" y1="8.382" x2="15" y2="8.27" width="0.254" layer="16"/>
-<via x="44.704" y="16.764" extent="1-16" drill="0.254"/>
-</signal>
-<signal name="N$3">
-<contactref element="R3" pad="2"/>
-</signal>
-<signal name="N$4">
-<via x="32" y="12" extent="1-16" drill="0.35"/>
-</signal>
-<signal name="N$22">
-<via x="35" y="34" extent="1-16" drill="0.35"/>
-</signal>
-<signal name="N$24">
-<via x="50" y="31" extent="1-16" drill="0.35"/>
+<wire x1="38.608" y1="10.414" x2="18" y2="10.414" width="0.3" layer="16"/>
+<wire x1="41.6" y1="18.2" x2="41.6" y2="14.4" width="0.3" layer="1"/>
+<wire x1="41.6" y1="14.4" x2="42" y2="14" width="0.3" layer="1"/>
+<via x="42" y="14" extent="1-16" drill="0.35"/>
+<wire x1="42" y1="14" x2="42" y2="13.806" width="0.3" layer="16"/>
+<wire x1="42" y1="13.806" x2="38.608" y2="10.414" width="0.3" layer="16"/>
+<wire x1="18" y1="10.414" x2="16.144" y2="12.27" width="0.3" layer="16"/>
+<wire x1="16.144" y1="12.27" x2="14" y2="12.27" width="0.3" layer="16"/>
 </signal>
 </signals>
