File: eagle/ver2_usb/team4-selo-atmega32u4-usb.sch (EAGLE design)
At the start: 35 parts, among them J1 3x2 M, J3 629105136821, SW2 !RESET, U3 ATMEGA32U4-AUR, X2 16 MHz

Commit message: add info to schematic
Other:
- note added: "SeLo I/O Control System"
Changed lines of the file:
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@@
 <text x="175.26" y="81.28" size="1.778" layer="97">D11#</text>
 <text x="175.26" y="78.74" size="1.778" layer="97">D12/A10</text>
+<wire x1="187.96" y1="127" x2="256.54" y2="127" width="0.1524" layer="97"/>
+<wire x1="256.54" y1="127" x2="256.54" y2="73.66" width="0.1524" layer="97"/>
+<wire x1="256.54" y1="73.66" x2="187.96" y2="73.66" width="0.1524" layer="97"/>
+<wire x1="187.96" y1="73.66" x2="187.96" y2="127" width="0.1524" layer="97"/>
+<text x="187.96" y="124.46" size="1.778" layer="97">SeLo I/O Control System</text>
 </plain>
 <instances>

Commit message: update board and schematic
Connections:
- removed net N$3: R3.2
- net VBUS: now also R3.2
Other:
- note added: "SeLo Security Locker An affordable, wall-mounted, and easy-to-use security locker that can be locked/unlocked using PINs and incorporate thief detection."
Changed lines of the file:
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@@
 <wire x1="187.96" y1="73.66" x2="187.96" y2="127" width="0.1524" layer="97"/>
 <text x="187.96" y="124.46" size="1.778" layer="97">SeLo I/O Control System</text>
+<text x="327.66" y="25.4" size="1.778" layer="97">SeLo Security Locker
+An affordable, wall-mounted, and easy-to-use security locker that can be locked/unlocked
+using PINs and incorporate thief detection.</text>
+<text x="339.852" y="7.112" size="2.54" layer="97">1</text>
 </plain>
 <instances>
@@
 <net name="VBUS" class="0">
 <segment>
-<wire x1="132.08" y1="111.76" x2="132.08" y2="109.22" width="0.1524" layer="91"/>
 <pinref part="U3" gate="G$1" pin="VBUS"/>
 <wire x1="132.08" y1="109.22" x2="137.16" y2="109.22" width="0.1524" layer="91"/>
@@
 <pinref part="VBUS6" gate="1" pin="VBUS"/>
 </segment>
+<segment>
+<wire x1="134.62" y1="153.67" x2="134.62" y2="152.4" width="0.1524" layer="91"/>
+<pinref part="R3" gate="G$1" pin="2"/>
+<pinref part="VBUS7" gate="1" pin="VBUS"/>
+<wire x1="134.62" y1="152.4" x2="134.62" y2="151.13" width="0.1524" layer="91"/>
+<wire x1="134.62" y1="154.94" x2="134.62" y2="153.67" width="0.1524" layer="91"/>
+</segment>
 </net>
 <net name="N$19" class="0">
@@
 </segment>
 </net>
-<net name="N$3" class="0">
-<segment>
-<wire x1="134.62" y1="153.67" x2="134.62" y2="151.13" width="0.1524" layer="91"/>
-<pinref part="R3" gate="G$1" pin="2"/>
-</segment>
-</net>
